File: hardware/SmartTBBatteryCharger.kicad_pcb (KiCad board)
At the start: 2 copper layers, 217 parts, among them J1 XT60_MALE, J2 XT60_MALE, J3 XT60_MALE, J4 XT60_MALE, J5 XT60_MALE, J6 XT60_MALE, J7 Conn_SWD, J8 Conn_01x02, Q1 BSC070N10NS5, Q2 BSC070N10NS5, Q3 BSC070N10NS5, Q4 BSC070N10NS5, Q5 BSC070N10NS5, Q6 BSC070N10NS5, U1 RY8411, U10 INA240A1PW, U11 UCC27517, U12 UCC27517, U13 UCC27517, U14 INA240A1PW, U15 INA240A1PW, U16 INA240A1PW, U2 RS3236, U3 RY8411, U4 STM32G474RBTx, U5 INA240A1PW, U6 UCC27517, U7 UCC27517, U8 INA240A1PW, U9 UCC27517, Y1 Crystal_GND24

Commit message: Update Hardware
Parts:
- moved C92 113.4 mm to (346.5, 58.2)
- moved C93 113.4 mm to (351.5, 58.2)
- moved D18 113.4 mm to (349.0, 58.0)
- moved D19 113.4 mm to (354.0, 58.0)
- moved C34 111.8 mm to (321.8, 40.9)
- moved C35 111.8 mm to (325.8, 35.9)
- moved C38 111.8 mm to (310.5, 34.5)
- moved C39 111.8 mm to (310.5, 37.0)
- moved R10 111.8 mm to (310.5, 44.5)
- moved R8 111.8 mm to (310.5, 39.5)
- moved R9 111.8 mm to (310.5, 42.0)
- moved C22 111.8 mm to (313.4, 47.4)
- moved C31 111.8 mm to (315.2, 42.0)
- moved C33 111.8 mm to (322.4, 47.4)
- moved C37 111.8 mm to (339.8, 34.8)
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Connections:
- C32 pad 1: Net-(D3-K) -> VPP
- C33 pad 1: Net-(D3-K) -> VPP
- C34 pad 1: Net-(D3-K) -> VPP
- C35 pad 1: Net-(D3-K) -> VPP
- C36 pad 1: Net-(D3-K) -> VPP
- C37 pad 1: Net-(D3-K) -> VPP
- D3 pad 1: Net-(D3-K) -> VPP
- J1 pad 2: Net-(D3-K) -> Net-(J1-Pin_2)
- R5 pad 1: Net-(D3-K) -> VPP
- R5 pad 2: Net-(U5-+) -> Net-(U5--)
- R5 pad 3: Net-(U5--) -> Net-(U5-+)
- R5 pad 4: VPP -> Net-(J1-Pin_2)

Commit message: Hardware Progress
Parts:
- removed C62, C63, C64, C65, C66, C67, C68, C70, C74, C78, C84, C85, C86: 100n, Capacitor_SMD:C_0603_1608Metric
- removed C69, C73, C77, C87, C88, C89: 100u, Capacitor_THT:CP_Radial_D6.3mm_P2.50mm
- removed C71, C72, C75, C76, C79, C80, C81, C82, C83: 10u, Capacitor_SMD:C_1206_3216Metric
- removed D10, D11, D9: K34, Diode_SMD:D_SOD-123F
- removed D12, D13, D14: SB1045, Diode_SMD:D_PowerDI-5
- removed F4, F5, F6: 8A, Fuse:Fuse_1206_3216Metric
- removed J4, J5, J6: XT60_MALE, Connector_AMASS:AMASS_XT60-M_1x02_P7.20mm_Vertical
- removed L6, L7, L8: 47u, Inductor_SMD:L_Coilcraft_MSS1260-XXX
- removed Q4, Q5, Q6: BSC070N10NS5, Package_TO_SOT_SMD:TDSON-8-1
- removed R21, R22, R23: 33R, Resistor_SMD:R_0603_1608Metric
- removed R24, R25, R26: 1R, Resistor_SMD:R_0603_1608Metric
- removed R27, R28, R29: 4m, Resistor_SMD:R_Shunt_Vishay_WSK2512_6332Metric_T1.19mm
- removed R30, R31, R32: 10k, Resistor_SMD:R_0603_1608Metric
- removed R33, R34, R35: 90k, Resistor_SMD:R_0603_1608Metric
- removed U11, U12, U13: UCC27517, Package_TO_SOT_SMD:SOT-23-5
- removed U14, U15, U16: INA240A1PW, Package_SO:TSSOP-8_4.4x3mm_P0.65mm
- added C104: 100u, Capacitor_THT:CP_Radial_D6.3mm_P2.50mm, F.Cu at (367.0, 32.3)
- C22, C31, C32, C33, C34, C42, C55, C58, D3, D4, D5, D6, D7, D8, Q1, Q2, Q3, R5, R6, U10, U5, U6, U7, U8, U9: moved to B.Cu
- C40, C41, C50, C51, C52, C61: value 100n -> 100u; footprint Capacitor_SMD:C_0603_1608Metric -> Capacitor_THT:CP_Radial_D6.3mm_P2.50mm
- C43: value 100u -> 10u; footprint Capacitor_THT:CP_Radial_D6.3mm_P2.50mm -> Capacitor_SMD:C_1206_3216Metric; moved to B.Cu
- C44, C54: value 100n -> 10u; footprint Capacitor_SMD:C_0603_1608Metric -> Capacitor_SMD:C_1206_3216Metric; moved to B.Cu
- C45, C47, C56: value 10u -> 100n; footprint Capacitor_SMD:C_1206_3216Metric -> Capacitor_SMD:C_0603_1608Metric; moved to B.Cu
- C46, C57: value 10u -> 100n; footprint Capacitor_SMD:C_1206_3216Metric -> Capacitor_SMD:C_0603_1608Metric
- C48: value 100n -> 10u; footprint Capacitor_SMD:C_0603_1608Metric -> Capacitor_SMD:C_1206_3216Metric
- C49: value 100u -> 100n; footprint Capacitor_THT:CP_Radial_D6.3mm_P2.50mm -> Capacitor_SMD:C_0603_1608Metric
- C53: value 100u -> 100n; footprint Capacitor_THT:CP_Radial_D6.3mm_P2.50mm -> Capacitor_SMD:C_0603_1608Metric; moved to B.Cu
- C59: value 100u -> 10u; footprint Capacitor_THT:CP_Radial_D6.3mm_P2.50mm -> Capacitor_SMD:C_1206_3216Metric
- R11, R16: value 33R -> 1R; moved to B.Cu
- R12, R17: value 1R -> 33R
- R13, R18: value 4m -> 10k; footprint Resistor_SMD:R_Shunt_Vishay_WSK2512_6332Metric_T1.19mm -> Resistor_SMD:R_0603_1608Metric
- R14, R19: value 10k -> 90k
- R15, R20: value 90k -> 4m; footprint Resistor_SMD:R_0603_1608Metric -> Resistor_SMD:R_Shunt_Vishay_WSK2512_6332Metric_T1.19mm; moved to B.Cu
- moved C60 214.8 mm to (399.3, 67.7), turned to 0 degrees
- moved R14 201.4 mm to (399.6, 51.8)
- moved R19 200.6 mm to (399.3, 75.2)
- moved R13 195.9 mm to (402.8, 45.0), turned to 90 degrees
- moved R18 192.3 mm to (399.3, 72.7), turned to 0 degrees
- moved R12 191.7 mm to (399.6, 49.2), turned to 0 degrees
- moved R17 191.5 mm to (399.3, 70.2), turned to 0 degrees
- moved C61 189.3 mm to (376.3, 64.5), turned to 0 degrees
- moved C46 189.1 mm to (399.6, 44.2), turned to 0 degrees
- moved R15 186.9 mm to (384.2, 43.0)
- moved R20 186.4 mm to (384.3, 64.2)
- moved C48 184.7 mm to (382.8, 44.0), turned to -90 degrees
- moved R11 183.2 mm to (381.5, 57.2), turned to -90 degrees
- moved R16 182.7 mm to (381.5, 78.5), turned to -90 degrees
- moved U7 179.3 mm to (384.5, 57.2), turned to 180 degrees
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Connections:
- C40 pad 1: +10V -> VPP
- C41 pad 1: GND -> VPP
- C41 pad 2: ISENSE_CH2 -> GND
- C42 pad 1: +3.3V -> VPP
- C43 pad 1: Net-(D6-K) -> VPP
- C44 pad 1: Net-(D6-K) -> VPP
- C45 pad 1: Net-(D6-K) -> +10V
- C46 pad 1: Net-(D6-K) -> GND
- C46 pad 2: GND -> ISENSE_CH2
- C47 pad 1: Net-(D6-K) -> +3.3V
- C47 pad 2: Net-(C47-Pad2) -> GND
- C48 pad 1: GND -> VPP
- C48 pad 2: VSENSE_CH2 -> Net-(C48-Pad2)
- C49 pad 1: Net-(D6-K) -> GND
- C49 pad 2: Net-(C47-Pad2) -> VSENSE_CH2
- C50 pad 1: +10V -> VPP
- C50 pad 2: GND -> Net-(C48-Pad2)
- C51 pad 1: GND -> VPP
- C51 pad 2: ISENSE_CH3 -> GND
- C52 pad 1: +3.3V -> VPP
- C53 pad 1: Net-(D8-K) -> VPP
- C54 pad 1: Net-(D8-K) -> VPP
- C55 pad 1: Net-(D8-K) -> VPP
- C56 pad 1: Net-(D8-K) -> +10V
- C57 pad 1: Net-(D8-K) -> GND
- C57 pad 2: Net-(C57-Pad2) -> ISENSE_CH3
- C58 pad 1: GND -> +3.3V
- C58 pad 2: VSENSE_CH3 -> GND
- C59 pad 1: Net-(D8-K) -> VPP
- C59 pad 2: Net-(C57-Pad2) -> Net-(C59-Pad2)
- C60 pad 1: +10V -> GND
- C60 pad 2: GND -> VSENSE_CH3
- C61 pad 1: +10V -> VPP
- C61 pad 2: GND -> Net-(C59-Pad2)
- D6 pad 1: Net-(D6-K) -> VPP
- D8 pad 1: Net-(D8-K) -> VPP
- F2 pad 2: Net-(C47-Pad2) -> Net-(C48-Pad2)
- F3 pad 2: Net-(C57-Pad2) -> Net-(C59-Pad2)
- J2 pad 2: Net-(D6-K) -> Net-(J2-Pin_2)
- J3 pad 2: Net-(D8-K) -> Net-(J3-Pin_2)
- L4 pad 2: Net-(C47-Pad2) -> Net-(C48-Pad2)
- L5 pad 2: Net-(C57-Pad2) -> Net-(C59-Pad2)
- R11 pad 1: ISENSE_CH2 -> Net-(D5-K)
- R11 pad 2: Net-(R11-Pad2) -> Net-(D5-A)
- R12 pad 1: Net-(D5-K) -> ISENSE_CH2
- R12 pad 2: Net-(D5-A) -> Net-(R12-Pad2)
- R13 pad 1: Net-(D6-K) -> GND
- R13 pad 2: Net-(U8-+) -> VSENSE_CH2
- R14 pad 1: GND -> VSENSE_CH2
- R14 pad 2: VSENSE_CH2 -> Net-(C48-Pad2)
- R15 pad 1: VSENSE_CH2 -> VPP
- R15 pad 2: Net-(C47-Pad2) -> Net-(U8--)
- R16 pad 1: ISENSE_CH3 -> Net-(D7-K)
- R16 pad 2: Net-(R16-Pad2) -> Net-(D7-A)
- R17 pad 1: Net-(D7-K) -> ISENSE_CH3
- R17 pad 2: Net-(D7-A) -> Net-(R17-Pad2)
- R18 pad 1: Net-(D8-K) -> GND
- R18 pad 2: Net-(U10-+) -> VSENSE_CH3
- R19 pad 1: GND -> VSENSE_CH3
- R19 pad 2: VSENSE_CH3 -> Net-(C59-Pad2)
- R20 pad 1: VSENSE_CH3 -> VPP
- R20 pad 2: Net-(C57-Pad2) -> Net-(U10--)
- U10 pad 8: Net-(R16-Pad2) -> Net-(R17-Pad2)
- U8 pad 8: Net-(R11-Pad2) -> Net-(R12-Pad2)
Routing:
- net Net-(U5-+): track 0.00 -> 17.6 mm
- net VPP: track 0.00 -> 17.4 mm
- net Net-(U5--): track 0.00 -> 13.3 mm
Other:
- board outline added: 100 x 100 mm
