File: hardware/SmartTBBatteryCharger.kicad_sch (KiCad schematic)
At the start: 217 parts, among them J1 XT60_MALE, J2 XT60_MALE, J3 XT60_MALE, J4 XT60_MALE, J5 XT60_MALE, J6 XT60_MALE, J7 Conn_SWD, J8 Conn_01x02, Q1 BSC070N10NS5, Q2 BSC070N10NS5, Q3 BSC070N10NS5, Q4 BSC070N10NS5, Q5 BSC070N10NS5, Q6 BSC070N10NS5, U1 RY8411, U10 INA240A1PW, U11 UCC27517, U12 UCC27517, U13 UCC27517, U14 INA240A1PW, U15 INA240A1PW, U16 INA240A1PW, U2 RS3236, U3 RY8411, U4 STM32G474RBTx, U5 INA240A1PW, U6 UCC27517, U7 UCC27517, U8 INA240A1PW, U9 UCC27517, Y1 Crystal_GND24

Commit message: Update Hardware
Connections:
- net VPP: now also C32.1, C33.1, C34.1, C35.1, C36.1, C37.1, D3.1 (K), R5.1; no longer R5.4
- net at U5.2 (+): now also R5.3; no longer R5.2
- net at U5.3 (-): now also R5.2; no longer R5.3
- new net: J1.2 (Pin_2), R5.4
Other:
- moved on the sheet: C22, C31, C32, C33, C34, C35, C36, C37, C38, C39, D3, D4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

Commit message: Hardware Progress
Parts:
- removed C40, C41, C50, C51, C52, C61, C62, C63, C64, C65, C66, C67, C68, C70, C74, C78, C84, C85, C86: 100n, Capacitor_SMD:C_0603_1608Metric, symbol Device:C
- removed C43, C49, C53, C59, C69, C73, C77, C87, C88, C89: 100u, Capacitor_THT:CP_Radial_D6.3mm_P2.50mm, symbol Device:C_Polarized
- removed C71, C72, C75, C76, C79, C80, C81, C82, C83: 10u, Capacitor_SMD:C_1206_3216Metric, symbol Device:C
- removed D10, D11, D9: K34, Diode_SMD:D_SOD-123F, symbol Device:D_Schottky
- removed D12, D13, D14: SB1045, Diode_SMD:D_PowerDI-5, symbol Device:D_Schottky
- removed F4, F5, F6: 8A, Fuse:Fuse_1206_3216Metric, symbol Device:Fuse
- removed J4, J5, J6: XT60_MALE, Connector_AMASS:AMASS_XT60-M_1x02_P7.20mm_Vertical, symbol Connector_Generic:Conn_01x02
- removed L6, L7, L8: 47u, Inductor_SMD:L_Coilcraft_MSS1260-XXX, symbol Device:L
- removed Q4, Q5, Q6: BSC070N10NS5, Package_TO_SOT_SMD:TDSON-8-1, symbol Transistor_FET:BSC070N10NS5
- removed R13, R18, R27, R28, R29: 4m, Resistor_SMD:R_Shunt_Vishay_WSK2512_6332Metric_T1.19mm, symbol Device:R_Shunt
- removed R15, R20, R33, R34, R35: 90k, Resistor_SMD:R_0603_1608Metric, symbol Device:R
- removed R21, R22, R23: 33R, Resistor_SMD:R_0603_1608Metric, symbol Device:R
- removed R24, R25, R26: 1R, Resistor_SMD:R_0603_1608Metric, symbol Device:R
- removed R30, R31, R32: 10k, Resistor_SMD:R_0603_1608Metric, symbol Device:R
- removed U11, U12, U13: UCC27517, Package_TO_SOT_SMD:SOT-23-5, symbol 0_RM2024:UCC27517
- removed U14, U15, U16: INA240A1PW, Package_SO:TSSOP-8_4.4x3mm_P0.65mm, symbol Amplifier_Current:INA240A1PW
- added C104, C40, C41, C50, C51, C52, C61: 100u, Capacitor_THT:CP_Radial_D6.3mm_P2.50mm, symbol Device:C_Polarized
- added C43, C59: 10u, Capacitor_SMD:C_1206_3216Metric, symbol Device:C
- added C49, C53: 100n, Capacitor_SMD:C_0603_1608Metric, symbol Device:C
- added R13, R18: 10k, Resistor_SMD:R_0603_1608Metric, symbol Device:R
- added R15, R20: 4m, Resistor_SMD:R_Shunt_Vishay_WSK2512_6332Metric_T1.19mm, symbol Device:R_Shunt
- C44, C48, C54: value 100n -> 10u; footprint Capacitor_SMD:C_0603_1608Metric -> Capacitor_SMD:C_1206_3216Metric
- C45, C46, C47, C56, C57: value 10u -> 100n; footprint Capacitor_SMD:C_1206_3216Metric -> Capacitor_SMD:C_0603_1608Metric
- R11, R16: value 33R -> 1R
- R12, R17: value 1R -> 33R
- R14, R19: value 10k -> 90k
Connections:
- net +10V: now also C45.1, C56.1; no longer C60.1
- net +3.3V: now also C47.1, C58.1; no longer C42.1
- net GND: now also C46.1, C47.2, C57.1, C58.2, C60.1, C104.2, C40.2, C41.2, C43.2, C49.1, C51.2, C52.2, C53.2, R13.1, R18.1; no longer C46.2, C48.1, C58.1, C60.2, R14.1, R19.1
- net ISENSE_CH2: now also C46.2, R12.1; no longer R11.1
- net ISENSE_CH3: now also C57.2, R17.1; no longer R16.1
- net VPP: now also C42.1, C44.1, C48.1, C54.1, C55.1, D6.1 (K), D8.1 (K), C104.1, C40.1, C41.1, C43.1, C50.1, C51.1, C52.1, C53.1, C59.1, C61.1, R15.1, R20.1
- net VSENSE_CH2: now also R14.1, C49.2, R13.2; no longer C48.2, R14.2
- net VSENSE_CH3: now also C60.2, R19.1, R18.2; no longer C58.2, R19.2
- net at U8.2 (+): now also R15.3
- net at U8.3 (-): now also R15.2
- net at R11.2: now also D5.2 (A), Q2.4 (G); no longer U8.8
- net at D7.1 (K), U9.5 (OUT): now also R16.1; no longer R17.1
- net at D7.2 (A), Q3.4 (G): now also R16.2; no longer R17.2
- net at U10.2 (+): now also R20.3
- net at U10.3 (-): now also R20.2
- net at F2.2, L4.2: now also C48.2, R14.2, C50.2; no longer C47.2
- net at U10.8: now also R17.2; no longer R16.2
- net at F3.2, L5.2: now also R19.2, C59.2, C61.2; no longer C57.2
- net at D5.1 (K), U7.5 (OUT): now also R11.1; no longer R12.1
- new net: J2.2 (Pin_2), R15.4
- new net: J3.2 (Pin_2), R20.4
- new net: R12.2, U8.8
Other:
- moved on the sheet: C35
