File: hardware_test_new_2/SmartTBBatteryChargerNewTest.kicad_pcb (KiCad board)
At the start: 4 copper layers, 81.6 x 48 mm, 161 parts, among them J1 XT60_MALE, J2 XT60_MALE, J7 Conn_SWD, J8 Conn_01x02, Q1 BSC070N10NS5, Q3 AO3400A, Q4 BSC070N10NS5, Q5 BSC070N10NS5, U1 RY8411, U10 UCC27201ADR, U2 RS3236, U3 RY8411, U4 STM32G474RBTx, U5 INA240A1PW, U6 UCC27517, U7 INA240A1PW, U9 INA240A1PW, Y3 CSTCE8M

Commit message: New test channel schematic
Parts:
- removed C100, C101, C102, C103, C31, C32, C38, C39, C58, C92, C93, C94, C95, C96, C97, C98, C99: 100n, Capacitor_SMD:C_0603_1608Metric
- removed C104, C35, C36, C42: 100u, Capacitor_THT:CP_Radial_D6.3mm_P2.50mm
- removed C33, C34, C37: 10u, Capacitor_SMD:C_1206_3216Metric
- removed D18, D19, D20, D21, D22, D23, D24, D25, D26, D27, D28, D29: WS2812B-2020, LED_SMD:LED_WS2812B-2020_PLCC4_2.0x2.0mm
- removed F1: 8A, Fuse:Fuse_1206_3216Metric
- removed F2: 5A, Fuse:Fuse_1206_3216Metric
- removed J1, J2: XT60_MALE, Connector_AMASS:AMASS_XT60-M_1x02_P7.20mm_Vertical
- removed L3: 47u, Inductor_SMD:L_Coilcraft_MSS1260-XXX
- removed Q1: BSC070N10NS5, Package_TO_SOT_SMD:TDSON-8-1
- removed R10: 90k, Resistor_SMD:R_0603_1608Metric
- removed R11, R8: 33R, Resistor_SMD:R_0603_1608Metric
- removed R12: 4m, Resistor_SMD:R_Shunt_Vishay_WSK2512_6332Metric_T1.19mm
- removed R9: 10k, Resistor_SMD:R_0603_1608Metric
- removed U10: UCC27201ADR, Package_SO:SOIC-8_3.9x4.9mm_P1.27mm
- removed U9: INA240A1PW, Package_SO:TSSOP-8_4.4x3mm_P0.65mm
- added C61: 10u, Capacitor_SMD:C_1206_3216Metric, F.Cu at (278.4, 74.9)
- added C62: 10n, Capacitor_SMD:C_0603_1608Metric, F.Cu at (290.9, 71.9)
- added C63: 10u, Capacitor_SMD:C_1206_3216Metric, F.Cu at (309.8, 71.5)
- added C64: 10u, Capacitor_SMD:C_1206_3216Metric, F.Cu at (309.8, 74.9)
- added D10: K34, Diode_SMD:D_SOD-123F, F.Cu at (188.3, 80.0)
- added D11: D_Schottky, Diode_SMD:D_PowerDI-5, F.Cu at (297.3, 92.0)
- added F3: 5A, Fuse:Fuse_1206_3216Metric, F.Cu at (284.1, 64.8)
- added F4: 5A, Fuse:Fuse_1206_3216Metric, F.Cu at (315.4, 64.8)
- added J3: XT60_MALE, Connector_AMASS:AMASS_XT30U-M_1x02_P5.0mm_Vertical, F.Cu at (268.5, 84.9)
- added J4: XT60_MALE, Connector_AMASS:AMASS_XT30U-M_1x02_P5.0mm_Vertical, F.Cu at (296.5, 80.8)
- added L5: 47u, Inductor_SMD:L_Coilcraft_MSS1260-XXX, F.Cu at (299.9, 70.3)
- added R33: 1R, Resistor_SMD:R_0603_1608Metric, F.Cu at (290.9, 79.5)
- added R34: 1k, Resistor_SMD:R_0603_1608Metric, F.Cu at (290.9, 82.0)
- C22, C49, C59: value 100n -> 10u; footprint Capacitor_SMD:C_0603_1608Metric -> Capacitor_SMD:C_1206_3216Metric; moved to F.Cu
- C24, C44, C50, C51, C52, R14, R15, R28: moved to F.Cu
- C41: value 100n -> 100u; footprint Capacitor_SMD:C_0603_1608Metric -> Capacitor_THT:CP_Radial_D6.3mm_P2.50mm; moved to F.Cu
- C47: value 10u -> 100n; footprint Capacitor_SMD:C_1206_3216Metric -> Capacitor_SMD:C_0603_1608Metric
- C48: value 100u -> 10u; footprint Capacitor_THT:CP_Radial_D6.3mm_P2.50mm -> Capacitor_SMD:C_1206_3216Metric; moved to F.Cu
- C60: value 100n -> 10n; moved to F.Cu
- D3: value SB1045 -> D_Schottky
- L4: moved to B.Cu
- R22: value 33R -> 10k; moved to F.Cu
- R23: value 4m -> 90k; footprint Resistor_SMD:R_Shunt_Vishay_WSK2512_6332Metric_T1.19mm -> Resistor_SMD:R_0603_1608Metric
- R29: value 1R -> 1k
- R5: value 4m -> 10m
- R6: value 1R -> 10m; footprint Resistor_SMD:R_0603_1608Metric -> Resistor_SMD:R_Shunt_Vishay_WSK2512_6332Metric_T1.19mm; moved to F.Cu
- U5, U7: value INA240A1PW -> INA180A1; footprint Package_SO:TSSOP-8_4.4x3mm_P0.65mm -> Package_TO_SOT_SMD:SOT-23-5; moved to F.Cu
- U6: value UCC27517 -> FD6288Q; footprint Package_TO_SOT_SMD:SOT-23-5 -> Package_DFN_QFN:QFN-24-1EP_4x4mm_P0.5mm_EP2.7x2.7mm; moved to F.Cu
- moved R22 238.1 mm to (290.9, 74.5), turned to 0 degrees
- moved C52 238.1 mm to (290.9, 69.4), turned to 0 degrees
- moved C51 233.8 mm to (290.9, 66.9), turned to 0 degrees
- moved Q5 228.6 mm to (309.2, 80.5)
- moved R23 227.5 mm to (290.9, 77.0), turned to 0 degrees
- moved C49 226.5 mm to (309.8, 68.2), turned to 0 degrees
- moved R6 219.5 mm to (297.8, 86.8), turned to 0 degrees
- moved U7 218.7 mm to (315.2, 68.8), turned to 0 degrees
- moved C41 212.5 mm to (307.9, 87.8)
- moved C48 211.7 mm to (309.8, 64.8), turned to 0 degrees
- moved C45 204.3 mm to (278.4, 64.8), turned to 0 degrees
- moved C46 203.6 mm to (278.4, 68.2), turned to 0 degrees
- moved C44 203.3 mm to (259.6, 66.9), turned to 0 degrees
- moved R15 198.3 mm to (259.6, 77.0), turned to 0 degrees
- moved C50 198.3 mm to (259.6, 69.4), turned to 0 degrees
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Connections:
- C22 pad 2: GNDPWR -> GND
- C24 pad 1: +10V -> Net-(D10-K)
- C24 pad 2: GNDPWR -> CHA_SW
- C41 pad 1: +3.3V -> VPP
- C41 pad 2: GND -> GNDPWR
- C44 pad 1: GND -> +3.3V
- C44 pad 2: ISENSE_CHA -> GND
- C47 pad 2: Net-(C47-Pad2) -> GNDPWR
- C48 pad 2: Net-(C47-Pad2) -> GNDPWR
- C49 pad 1: SW_A -> VPP
- C49 pad 2: Net-(U10-HB) -> GNDPWR
- C50 pad 2: VSENSE_CHA -> /ChannelA1/CH_VSENSE
- C52 pad 2: ISENSE_INPUT -> /ChannelA2/CH_VSENSE
- C59 pad 1: +3.3V -> Net-(C59-Pad1)
- C59 pad 2: GND -> GNDPWR
- C60 pad 1: +3.3V -> /ChannelA1/CH_ISENSE
- D3 pad 1: VPP -> /ChannelA1/CH_SW
- D3 pad 2: Net-(D3-A) -> GNDPWR
- F8 pad 1: Net-(F8-Pad1) -> VPP
- L4 pad 1: SW_A -> /ChannelA1/CH_SW
- L4 pad 2: Net-(C47-Pad2) -> Net-(C59-Pad1)
- Q4 pad 1: SW_A -> /ChannelA1/CH_SW
- Q4 pad 2: SW_A -> /ChannelA1/CH_SW
- Q4 pad 3: SW_A -> /ChannelA1/CH_SW
- Q5 pad 1: GNDPWR -> /ChannelA2/CH_SW
- Q5 pad 2: GNDPWR -> /ChannelA2/CH_SW
- Q5 pad 3: GNDPWR -> /ChannelA2/CH_SW
- Q5 pad 5: SW_A -> VPP
- R14 pad 2: VSENSE_CHA -> /ChannelA1/CH_VSENSE
- R15 pad 1: VSENSE_CHA -> /ChannelA1/CH_VSENSE
- R15 pad 2: Net-(C47-Pad2) -> /ChannelA1/CH_VOUT
- R22 pad 1: ISENSE_INPUT -> GND
- R22 pad 2: Net-(R22-Pad2) -> /ChannelA2/CH_VSENSE
- R23 pad 1: Net-(F8-Pad1) -> /ChannelA2/CH_VSENSE
- R23 pad 2: Net-(U9--) -> /ChannelA2/CH_VOUT
- R28 pad 1: Net-(U10-HO) -> /ChannelA1/CH_HG
- R29 pad 1: Net-(U10-LO) -> Net-(R29-Pad1)
- R29 pad 2: Net-(Q5-G) -> /ChannelA1/CH_ISENSE
- R5 pad 1: VPP -> Net-(J3-Pin_1)
- R5 pad 2: Net-(U5--) -> CHA_SHUNT+
- R5 pad 3: Net-(U5-+) -> CHA_SHUNT-
- R5 pad 4: Net-(J1-Pin_2) -> GNDPWR
- R6 pad 1: Net-(U6-OUT) -> Net-(J4-Pin_1)
- R6 pad 2: Net-(Q1-G) -> CHA_SHUNT+
- U5 pad 1: GND -> Net-(R29-Pad1)
- U5 pad 2: Net-(U5-+) -> GND
- U5 pad 3: Net-(U5--) -> /ChannelA1/CH_SHUNT+
- U5 pad 4: GND -> /ChannelA1/CH_SHUNT-
- U6 pad 1: +10V -> unconnected-(U6-LIN1-Pad1)
- U6 pad 2: GNDPWR -> unconnected-(U6-LIN2-Pad2)
- U6 pad 3: DRV_CHB -> unconnected-(U6-LIN3-Pad3)
- U6 pad 4: GNDPWR -> +10V
- U6 pad 5: Net-(U6-OUT) -> unconnected-(U6-NC-Pad5)
- U7 pad 1: GND -> Net-(R34-Pad1)
- U7 pad 2: Net-(U7-+) -> GND
- U7 pad 3: Net-(U7--) -> /ChannelA2/CH_SHUNT+
- U7 pad 4: GND -> /ChannelA2/CH_SHUNT-
Routing:
- net +3.3V: track 194.7 -> 0.00 mm, vias 43 -> 0
- net VPP: track 169.7 -> 0.00 mm, vias 1 -> 0
- net +10V: track 129.0 -> 0.00 mm, vias 2 -> 0
- net RGB_DATA: track 121.7 -> 0.00 mm
- net +5V: track 94.7 -> 0.00 mm, vias 5 -> 0
- net Net-(R11-Pad2): track 78.1 -> 0.00 mm
- net Net-(C36-Pad2): track 72.8 -> 0.00 mm, vias 1 -> 0
- net Net-(R8-Pad2): track 64.0 -> 0.00 mm
- net DRV_CHB: track 58.4 -> 0.00 mm
- net DRV_CHA1: track 49.1 -> 0.00 mm
- net DRV_CHA2: track 48.4 -> 0.00 mm
- net Net-(C47-Pad2): track 47.2 -> 0.00 mm, vias 1 -> 0
- net GND: track 22.6 -> 0.00 mm, vias 656 -> 0
- net Net-(BZ1-+): track 19.2 -> 0.00 mm
- net GNDPWR: track 19.0 -> 0.00 mm, vias 142 -> 0
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- removed copper zone on B.Cu, net +10V
- removed copper zone on B.Cu, net +3.3V
- removed copper zone on B.Cu, net +5V
- removed copper zone on F.Cu, net +5V
- removed copper zone on In2.Cu, net GND
- removed copper zone on B.Cu, net GNDPWR
- removed copper zone on F.Cu, net GNDPWR
- removed copper zone on In1.Cu, net GNDPWR
- removed copper zone on In2.Cu, net GNDPWR
- removed copper zone on F.Cu, net Net-(C36-Pad2)
- removed copper zone on F.Cu, net Net-(C47-Pad2)
- removed copper zone on F.Cu, net Net-(D3-A)
- removed copper zone on F.Cu, net Net-(F8-Pad1)
- removed copper zone on F.Cu, net Net-(J1-Pin_1)
- removed copper zone on B.Cu, net Net-(J7-Pin_4)
- removed copper zone on F.Cu, net Net-(J7-Pin_4)
- removed copper zone on F.Cu, net Net-(J8-Pin_2)
- removed copper zone on B.Cu, net Net-(U1-LX)
- removed copper zone on B.Cu, net Net-(U3-LX)
- removed copper zone on F.Cu, net SW_A
- removed copper zone on B.Cu, net VPP
- removed copper zone on F.Cu, net VPP
Other:
- board outline removed
- board text removed: "SmartTBCharger V0.1 By RY RM2024"

Commit message: test2 schematic
Parts:
- added C100: 100n, Capacitor_SMD:C_0603_1608Metric, F.Cu at (213.9, 130.9)
- added C42: 100u, Capacitor_THT:CP_Radial_D6.3mm_P2.50mm, B.Cu at (222.6, 90.5)
- added C58: 100n, Capacitor_SMD:C_0603_1608Metric, F.Cu at (228.6, 90.0)
- added C65: 10u, Capacitor_SMD:C_1206_3216Metric, F.Cu at (224.5, 92.3)
- added C66: 10u, Capacitor_SMD:C_1206_3216Metric, F.Cu at (227.9, 91.8)
- added C67: 100n, Capacitor_SMD:C_0603_1608Metric, F.Cu at (230.2, 95.1)
- added C68: 10n, Capacitor_SMD:C_0603_1608Metric, F.Cu at (207.2, 91.0)
- added C69: 10u, Capacitor_SMD:C_1206_3216Metric, F.Cu at (238.0, 88.3)
- added C70: 10u, Capacitor_SMD:C_1206_3216Metric, F.Cu at (238.0, 90.7)
- added C71: 100n, Capacitor_SMD:C_0603_1608Metric, F.Cu at (213.9, 87.8)
- added C72: 100u, Capacitor_THT:CP_Radial_D6.3mm_P2.50mm, B.Cu at (222.6, 104.9)
- added C73: 100u, Capacitor_THT:CP_Radial_D6.3mm_P2.50mm, B.Cu at (222.6, 119.2)
- added C74: 100u, Capacitor_THT:CP_Radial_D6.3mm_P2.50mm, B.Cu at (222.6, 133.6)
- added C75: 100n, Capacitor_SMD:C_0603_1608Metric, F.Cu at (228.6, 104.3)
- added C76: 100n, Capacitor_SMD:C_0603_1608Metric, F.Cu at (228.6, 118.7)
- added C77: 100n, Capacitor_SMD:C_0603_1608Metric, F.Cu at (228.6, 133.1)
- added C78: 10u, Capacitor_SMD:C_1206_3216Metric, F.Cu at (227.9, 106.1)
- added C79: 10u, Capacitor_SMD:C_1206_3216Metric, F.Cu at (224.5, 121.0)
- added C80: 10u, Capacitor_SMD:C_1206_3216Metric, F.Cu at (227.9, 134.9)
- added C81: 10u, Capacitor_SMD:C_1206_3216Metric, F.Cu at (224.5, 106.6)
- added C82: 10u, Capacitor_SMD:C_1206_3216Metric, F.Cu at (227.9, 120.5)
- added C83: 10u, Capacitor_SMD:C_1206_3216Metric, F.Cu at (224.5, 135.4)
- added C84: 100n, Capacitor_SMD:C_0603_1608Metric, F.Cu at (230.2, 109.4)
- added C85: 100n, Capacitor_SMD:C_0603_1608Metric, F.Cu at (230.2, 123.8)
- added C86: 100n, Capacitor_SMD:C_0603_1608Metric, F.Cu at (230.2, 138.2)
- added C87: 10n, Capacitor_SMD:C_0603_1608Metric, F.Cu at (207.2, 105.3)
- added C88: 10n, Capacitor_SMD:C_0603_1608Metric, F.Cu at (207.2, 119.7)
- added C89: 10n, Capacitor_SMD:C_0603_1608Metric, F.Cu at (207.2, 134.1)
- added C92: 10u, Capacitor_SMD:C_1206_3216Metric, F.Cu at (238.0, 131.4)
- added C93: 10u, Capacitor_SMD:C_1206_3216Metric, F.Cu at (238.0, 119.4)
- added C94: 10u, Capacitor_SMD:C_1206_3216Metric, F.Cu at (238.0, 102.6)
- added C95: 10u, Capacitor_SMD:C_1206_3216Metric, F.Cu at (238.0, 105.0)
- added C96: 10u, Capacitor_SMD:C_1206_3216Metric, F.Cu at (238.0, 117.0)
- added C97: 10u, Capacitor_SMD:C_1206_3216Metric, F.Cu at (238.0, 133.8)
- added C98: 100n, Capacitor_SMD:C_0603_1608Metric, F.Cu at (213.9, 102.1)
- added C99: 100n, Capacitor_SMD:C_0603_1608Metric, F.Cu at (213.8, 116.5)
- added D12: D_Schottky, Diode_SMD:D_PowerDI-5, F.Cu at (232.4, 89.3)
- added D13: D_Schottky, Diode_SMD:D_PowerDI-5, F.Cu at (232.4, 103.6)
- added D14: D_Schottky, Diode_SMD:D_PowerDI-5, F.Cu at (232.4, 118.0)
- added D16: D_Schottky, Diode_SMD:D_PowerDI-5, F.Cu at (232.4, 132.4)
- added F10: 5A, Fuse:Fuse_1206_3216Metric, F.Cu at (239.7, 129.0)
- added F5: 5A, Fuse:Fuse_1206_3216Metric, F.Cu at (239.7, 85.9)
- added F6: 5A, Fuse:Fuse_1206_3216Metric, F.Cu at (239.7, 100.2)
- added F9: 5A, Fuse:Fuse_1206_3216Metric, F.Cu at (239.7, 114.6)
- added J10: XT60_MALE, Connector_AMASS:AMASS_XT30U-M_1x02_P5.0mm_Vertical, F.Cu at (246.7, 134.7)
- added J5: XT60_MALE, Connector_AMASS:AMASS_XT30U-M_1x02_P5.0mm_Vertical, F.Cu at (246.7, 91.6)
- added J6: XT60_MALE, Connector_AMASS:AMASS_XT30U-M_1x02_P5.0mm_Vertical, F.Cu at (246.7, 105.9)
- added J9: XT60_MALE, Connector_AMASS:AMASS_XT30U-M_1x02_P5.0mm_Vertical, F.Cu at (246.7, 120.3)
- added L6: 47u, Inductor_SMD:L_Coilcraft_MSS1260-XXX, B.Cu at (235.1, 88.6)
- added L7: 47u, Inductor_SMD:L_Coilcraft_MSS1260-XXX, B.Cu at (235.1, 103.0)
- added L8: 47u, Inductor_SMD:L_Coilcraft_MSS1260-XXX, B.Cu at (235.1, 117.4)
- added L9: 47u, Inductor_SMD:L_Coilcraft_MSS1260-XXX, B.Cu at (235.1, 131.7)
- added Q6: BSC070N10NS5, Package_TO_SOT_SMD:TDSON-8-1, F.Cu at (226.3, 86.6)
- added Q7: BSC070N10NS5, Package_TO_SOT_SMD:TDSON-8-1, F.Cu at (226.3, 100.9)
- added Q8: BSC070N10NS5, Package_TO_SOT_SMD:TDSON-8-1, F.Cu at (226.3, 115.3)
- added Q9: BSC070N10NS5, Package_TO_SOT_SMD:TDSON-8-1, F.Cu at (226.3, 129.7)
- added R10: 10m, Resistor_SMD:R_Shunt_Vishay_WSK2512_6332Metric_T1.19mm, F.Cu at (239.1, 122.6)
- added R11: 10m, Resistor_SMD:R_Shunt_Vishay_WSK2512_6332Metric_T1.19mm, F.Cu at (239.1, 137.0)
- added R35: 1R, Resistor_SMD:R_0603_1608Metric, F.Cu at (207.2, 87.7)
- added R38: 1k, Resistor_SMD:R_0603_1608Metric, F.Cu at (207.2, 93.5)
- added R39: 10k, Resistor_SMD:R_0603_1608Metric, F.Cu at (213.9, 90.3)
- added R40: 90k, Resistor_SMD:R_0603_1608Metric, F.Cu at (213.9, 92.8)
- added R41: 1R, Resistor_SMD:R_0603_1608Metric, F.Cu at (207.2, 102.0)
- added R42: 1R, Resistor_SMD:R_0603_1608Metric, F.Cu at (207.2, 116.4)
- added R43: 1R, Resistor_SMD:R_0603_1608Metric, F.Cu at (207.2, 130.8)
- added R44: 1k, Resistor_SMD:R_0603_1608Metric, F.Cu at (207.2, 107.8)
- added R45: 1k, Resistor_SMD:R_0603_1608Metric, F.Cu at (207.2, 122.2)
- added R46: 1k, Resistor_SMD:R_0603_1608Metric, F.Cu at (207.2, 136.6)
- added R47: 10k, Resistor_SMD:R_0603_1608Metric, F.Cu at (213.9, 104.6)
- added R48: 10k, Resistor_SMD:R_0603_1608Metric, F.Cu at (213.8, 119.0)
- added R49: 10k, Resistor_SMD:R_0603_1608Metric, F.Cu at (213.9, 133.4)
- added R50: 90k, Resistor_SMD:R_0603_1608Metric, F.Cu at (213.9, 107.1)
- added R51: 90k, Resistor_SMD:R_0603_1608Metric, F.Cu at (213.8, 121.5)
- added R52: 90k, Resistor_SMD:R_0603_1608Metric, F.Cu at (213.9, 135.9)
- added R8: 10m, Resistor_SMD:R_Shunt_Vishay_WSK2512_6332Metric_T1.19mm, F.Cu at (239.1, 93.9)
- added R9: 10m, Resistor_SMD:R_Shunt_Vishay_WSK2512_6332Metric_T1.19mm, F.Cu at (239.1, 108.2)
- added U10: INA180A1, Package_TO_SOT_SMD:SOT-23-5, F.Cu at (232.7, 124.4)
- added U11: INA180A1, Package_TO_SOT_SMD:SOT-23-5, F.Cu at (232.7, 138.8)
- added U8: INA180A1, Package_TO_SOT_SMD:SOT-23-5, F.Cu at (232.7, 95.7)
- added U9: INA180A1, Package_TO_SOT_SMD:SOT-23-5, F.Cu at (232.7, 110.0)
- C41, L5: moved to B.Cu
- moved C41 86.1 mm to (222.6, 76.3), turned to -90 degrees
- moved C49 85.8 mm to (224.5, 78.1), turned to -90 degrees
- moved R33 83.9 mm to (207.2, 73.5)
- moved C62 83.8 mm to (207.2, 76.8)
- moved R34 83.7 mm to (207.2, 79.3)
- moved U7 83.4 mm to (232.7, 81.5), turned to 90 degrees
- moved Q5 83.3 mm to (226.3, 72.4), turned to 180 degrees
- moved C48 82.8 mm to (227.9, 77.6)
- moved C52 77.1 mm to (213.9, 73.5)
- moved R22 77.0 mm to (213.9, 76.1)
- moved R23 77.0 mm to (213.9, 78.6)
- moved F4 76.0 mm to (239.7, 71.7), turned to 180 degrees
- moved C63 71.8 mm to (238.0, 74.1), turned to 180 degrees
- moved C64 71.8 mm to (238.0, 76.5), turned to 180 degrees
- moved D11 67.0 mm to (232.4, 75.1), turned to -90 degrees
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Connections:
- R5 pad 2: CHA_SHUNT+ -> /ChannelA1/CH_SHUNT+
- R5 pad 3: CHA_SHUNT- -> /ChannelA1/CH_SHUNT-
- R6 pad 2: CHA_SHUNT+ -> /ChannelA2/CH_SHUNT+
- R6 pad 3: CHA_SHUNT- -> /ChannelA2/CH_SHUNT-
Routing:
- net /ChannelA1/CH_SHUNT+: track 0.00 -> 10.6 mm
- net /ChannelC2/CH_SHUNT+: track 0.00 -> 10.6 mm
- net /ChannelB1/CH_SHUNT+: track 0.00 -> 10.6 mm
- net /ChannelA2/CH_SHUNT+: track 0.00 -> 10.6 mm
- net /ChannelC1/CH_SHUNT+: track 0.00 -> 10.6 mm
- net /ChannelB2/CH_SHUNT+: track 0.00 -> 10.6 mm
- net /ChannelC1/CH_SHUNT-: track 0.00 -> 7.81 mm
- net /ChannelB2/CH_SHUNT-: track 0.00 -> 7.81 mm
- net /ChannelB1/CH_SHUNT-: track 0.00 -> 7.81 mm
- net /ChannelA2/CH_SHUNT-: track 0.00 -> 7.81 mm
- net /ChannelA1/CH_SHUNT-: track 0.00 -> 7.81 mm
- net /ChannelC2/CH_SHUNT-: track 0.00 -> 7.81 mm

Commit message: test2 schematic should ok
Parts:
- removed Y3: CSTCE8M, Crystal:Resonator_SMD_Murata_CSTxExxV-3Pin_3.0x1.1mm_HandSoldering
- added C101: 100n, Capacitor_SMD:C_0603_1608Metric, F.Cu at (99.4, 58.8)
- added C102: 100n, Capacitor_SMD:C_0603_1608Metric, F.Cu at (103.4, 38.7)
- added C103: 100n, Capacitor_SMD:C_0603_1608Metric, F.Cu at (103.4, 41.2)
- added C104: 100n, Capacitor_SMD:C_0603_1608Metric, F.Cu at (103.4, 43.8)
- added C105: 100n, Capacitor_SMD:C_0603_1608Metric, F.Cu at (103.4, 46.3)
- added C106: 100n, Capacitor_SMD:C_0603_1608Metric, F.Cu at (103.4, 48.8)
- added C107: 100n, Capacitor_SMD:C_0603_1608Metric, F.Cu at (103.4, 51.3)
- added C108: 100n, Capacitor_SMD:C_0603_1608Metric, F.Cu at (103.4, 53.8)
- added C109: 100n, Capacitor_SMD:C_0603_1608Metric, F.Cu at (103.4, 56.3)
- added C110: 100n, Capacitor_SMD:C_0603_1608Metric, F.Cu at (190.9, 71.9)
- added C111: 100n, Capacitor_SMD:C_0603_1608Metric, F.Cu at (122.6, 76.7)
- added C31: 100n, Capacitor_SMD:C_0603_1608Metric, F.Cu at (197.8, 69.9)
- added C32: 100n, Capacitor_SMD:C_0603_1608Metric, F.Cu at (197.8, 72.9)
- added C33: 10u, Capacitor_SMD:C_1206_3216Metric, F.Cu at (109.7, 72.8)
- added C34: 100n, Capacitor_SMD:C_0603_1608Metric, F.Cu at (99.4, 43.8)
- added C35: 100n, Capacitor_SMD:C_0603_1608Metric, F.Cu at (99.4, 46.3)
- added C36: 100n, Capacitor_SMD:C_0603_1608Metric, F.Cu at (99.4, 48.8)
- added C37: 100n, Capacitor_SMD:C_0603_1608Metric, F.Cu at (99.4, 51.3)
- added C38: 100n, Capacitor_SMD:C_0603_1608Metric, F.Cu at (99.4, 53.8)
- added C39: 100n, Capacitor_SMD:C_0603_1608Metric, F.Cu at (99.4, 56.3)
- added D18: K34, Diode_SMD:D_SOD-123F, B.Cu at (199.7, 69.5)
- added D19: K34, Diode_SMD:D_SOD-123F, B.Cu at (199.7, 72.1)
- added D20: K34, Diode_SMD:D_SOD-123F, F.Cu at (100.1, 68.4)
- added D21: K34, Diode_SMD:D_SOD-123F, F.Cu at (100.1, 71.8)
- added D22: K34, Diode_SMD:D_SOD-123F, F.Cu at (100.1, 75.1)
- added D23: LED_BLUE, LED_SMD:LED_0603_1608Metric, F.Cu at (104.9, 61.4)
- added D24: LED_BLUE, LED_SMD:LED_0603_1608Metric, F.Cu at (104.9, 64.0)
- added D25: LED_BLUE, LED_SMD:LED_0603_1608Metric, F.Cu at (104.9, 66.5)
- added D26: LED_BLUE, LED_SMD:LED_0603_1608Metric, F.Cu at (104.9, 69.1)
- added D27: LED_BLUE, LED_SMD:LED_0603_1608Metric, F.Cu at (104.9, 71.7)
- added D28: LED_BLUE, LED_SMD:LED_0603_1608Metric, F.Cu at (104.9, 74.3)
- added D29: WS2812B, LED_SMD:LED_WS2812B_PLCC4_5.0x5.0mm_P3.2mm, F.Cu at (93.3, 60.6)
- added D30: WS2812B, LED_SMD:LED_WS2812B_PLCC4_5.0x5.0mm_P3.2mm, F.Cu at (93.3, 67.3)
- added D31: WS2812B, LED_SMD:LED_WS2812B_PLCC4_5.0x5.0mm_P3.2mm, F.Cu at (93.3, 73.9)
- added R12: 10k, Resistor_SMD:R_0603_1608Metric, F.Cu at (103.4, 58.8)
- added R53: 33, Resistor_SMD:R_0603_1608Metric, F.Cu at (107.4, 53.8)
- added R54: 10k, Resistor_SMD:R_0603_1608Metric, F.Cu at (107.4, 56.3)
- added R55: 33, Resistor_SMD:R_0603_1608Metric, F.Cu at (107.4, 58.8)
- added R56: 10k, Resistor_SMD:R_0603_1608Metric, F.Cu at (111.4, 38.7)
- added R57: 33, Resistor_SMD:R_0603_1608Metric, F.Cu at (111.4, 41.2)
- added R58: 2.2k, Resistor_SMD:R_0603_1608Metric, F.Cu at (111.4, 43.8)
- added R59: 2.2k, Resistor_SMD:R_0603_1608Metric, F.Cu at (111.4, 46.3)
- added R60: 2.2k, Resistor_SMD:R_0603_1608Metric, F.Cu at (111.4, 48.8)
- added R61: 2.2k, Resistor_SMD:R_0603_1608Metric, F.Cu at (111.4, 51.3)
- added R62: 2.2k, Resistor_SMD:R_0603_1608Metric, F.Cu at (111.4, 53.8)
- added R63: 2.2k, Resistor_SMD:R_0603_1608Metric, F.Cu at (111.4, 56.3)
- added R64: 33, Resistor_SMD:R_0603_1608Metric, F.Cu at (111.4, 58.8)
- added RN1: R_Pack04, Resistor_SMD:R_Array_Convex_4x0603, F.Cu at (109.0, 62.4)
- added RN2: R_Pack04, Resistor_SMD:R_Array_Convex_4x0603, F.Cu at (192.9, 66.6)
- added SW1: SW_Push, Button_Switch_SMD:SW_SPST_SKQG_WithStem, F.Cu at (84.5, 40.9)
- added SW2: SW_Push, Button_Switch_SMD:SW_SPST_SKQG_WithStem, F.Cu at (84.5, 47.6)
- added SW3: SW_Push, Button_Switch_SMD:SW_SPST_SKQG_WithStem, F.Cu at (84.5, 54.4)
- added SW4: SW_Push, Button_Switch_SMD:SW_SPST_SKQG_WithStem, F.Cu at (84.5, 61.1)
- added SW5: SW_Push, Button_Switch_SMD:SW_SPST_SKQG_WithStem, F.Cu at (84.5, 67.8)
- added SW6: SW_Push, Button_Switch_SMD:SW_SPST_SKQG_WithStem, F.Cu at (84.5, 74.6)
- added U12: FD6288Q, Package_DFN_QFN:QFN-24-1EP_4x4mm_P0.5mm_EP2.7x2.7mm, F.Cu at (110.1, 68.0)
- D10: moved to B.Cu
- D4, D5, D6: value LED -> WS2812B; footprint LED_SMD:LED_0603_1608Metric -> LED_SMD:LED_WS2812B_PLCC4_5.0x5.0mm_P3.2mm
- J8: footprint Connector_AMASS:AMASS_XT30U-M_1x02_P5.0mm_Vertical -> Connector_AMASS:AMASS_XT60-M_1x02_P7.20mm_Vertical
- R13, R17: value 33r -> 33; moved to F.Cu
- R16: value 33r -> 10k; moved to F.Cu
- R3: value 53.6k -> 54.7k
- R30, R32: value 2.2k -> 10k
- R31: value 2.2k -> 33
- moved R13 54.4 mm to (107.4, 38.7), turned to 0 degrees
- moved R17 54.0 mm to (107.4, 43.8), turned to 0 degrees
- moved R32 52.2 mm to (107.4, 51.3), turned to 0 degrees
- moved R16 52.1 mm to (107.4, 41.2), turned to 0 degrees
- moved R31 51.2 mm to (107.4, 48.8), turned to 0 degrees
- moved R30 50.4 mm to (107.4, 46.3), turned to 0 degrees
- moved D4 33.8 mm to (93.3, 40.8), turned to 0 degrees
- moved D5 32.3 mm to (93.3, 47.4), turned to 0 degrees
- moved D6 30.5 mm to (93.3, 54.0), turned to 0 degrees
- moved D10 25.2 mm to (199.7, 67.1), turned to 0 degrees
- moved C24 23.3 mm to (196.3, 67.3)
- moved U6 23.1 mm to (194.4, 70.8)
- moved C22 22.4 mm to (189.0, 71.3)
- moved C78 3.44 mm to (224.5, 106.6), turned to -90 degrees
- moved C81 3.44 mm to (227.9, 106.1), turned to 0 degrees
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Connections:
- net /ChannelB2/CH_SW renamed CHB2_SW
- net /ChannelC1/CH_SW renamed CHC1_SW
- net /ChannelC2/CH_SW renamed CHC2_SW
- C100 pad 2: /ChannelC2/CH_VSENSE -> CHC2_VS
- C24 pad 2: CHA_SW -> CHA1_SW
- C50 pad 2: /ChannelA1/CH_VSENSE -> CHA1_VS
- C52 pad 2: /ChannelA2/CH_VSENSE -> CHA2_VS
- C60 pad 1: /ChannelA1/CH_ISENSE -> CHA1_IS
- C62 pad 1: /ChannelA2/CH_ISENSE -> CHA2_IS
- C68 pad 1: /ChannelB1/CH_ISENSE -> CHB1_IS
- C71 pad 2: /ChannelB1/CH_VSENSE -> CHB1_VS
- C87 pad 1: /ChannelB2/CH_ISENSE -> CHB2_IS
- C88 pad 1: /ChannelC1/CH_ISENSE -> CHC1_IS
- C89 pad 1: /ChannelC2/CH_ISENSE -> CHC2_IS
- C98 pad 2: /ChannelB2/CH_VSENSE -> CHB2_VS
- C99 pad 2: /ChannelC1/CH_VSENSE -> CHC1_VS
- D11 pad 1: /ChannelA2/CH_SW -> CHA2_SW
- D12 pad 1: /ChannelB1/CH_SW -> CHB1_SW
- D3 pad 1: /ChannelA1/CH_SW -> CHA1_SW
- D4 pad 1: GND -> +5V
- D4 pad 2: Net-(D4-A) -> Net-(D4-DOUT)
- D5 pad 1: GND -> +5V
- D5 pad 2: Net-(D5-A) -> Net-(D5-DOUT)
- D6 pad 1: GND -> +5V
- D6 pad 2: Net-(D6-A) -> Net-(D29-DIN)
- L4 pad 1: /ChannelA1/CH_SW -> CHA1_SW
- L5 pad 1: /ChannelA2/CH_SW -> CHA2_SW
- L6 pad 1: /ChannelB1/CH_SW -> CHB1_SW
- Q4 pad 1: /ChannelA1/CH_SW -> CHA1_SW
- Q4 pad 2: /ChannelA1/CH_SW -> CHA1_SW
- Q4 pad 3: /ChannelA1/CH_SW -> CHA1_SW
- Q5 pad 1: /ChannelA2/CH_SW -> CHA2_SW
- Q5 pad 2: /ChannelA2/CH_SW -> CHA2_SW
- Q5 pad 3: /ChannelA2/CH_SW -> CHA2_SW
- Q6 pad 1: /ChannelB1/CH_SW -> CHB1_SW
- Q6 pad 2: /ChannelB1/CH_SW -> CHB1_SW
- Q6 pad 3: /ChannelB1/CH_SW -> CHB1_SW
- R13 pad 1: DRV_CHA2 -> BTN1
- R13 pad 2: Net-(U4-PA9) -> Net-(R12-Pad2)
- R14 pad 2: /ChannelA1/CH_VSENSE -> CHA1_VS
- R15 pad 1: /ChannelA1/CH_VSENSE -> CHA1_VS
- R16 pad 1: DRV_CHA1 -> +3.3V
- R16 pad 2: Net-(U4-PA8) -> Net-(R16-Pad2)
- R17 pad 1: DRV_CHB -> BTN2
- R17 pad 2: Net-(U4-PA10) -> Net-(R16-Pad2)
- R22 pad 2: /ChannelA2/CH_VSENSE -> CHA2_VS
- R23 pad 1: /ChannelA2/CH_VSENSE -> CHA2_VS
- R28 pad 1: /ChannelA1/CH_HG -> CHA1_HG
- R29 pad 2: /ChannelA1/CH_ISENSE -> CHA1_IS
- R30 pad 1: Net-(U4-PA8) -> +3.3V
- R30 pad 2: Net-(D5-A) -> Net-(R30-Pad2)
- R31 pad 1: Net-(U4-PA9) -> BTN3
- R31 pad 2: Net-(D6-A) -> Net-(R30-Pad2)
- R32 pad 1: Net-(U4-PA10) -> +3.3V
- R32 pad 2: Net-(D4-A) -> Net-(R32-Pad2)
- R33 pad 1: /ChannelA2/CH_HG -> CHA2_HG
- R34 pad 2: /ChannelA2/CH_ISENSE -> CHA2_IS
- R35 pad 1: /ChannelB1/CH_HG -> CHB1_HG
- R38 pad 2: /ChannelB1/CH_ISENSE -> CHB1_IS
- R39 pad 2: /ChannelB1/CH_VSENSE -> CHB1_VS
- R40 pad 1: /ChannelB1/CH_VSENSE -> CHB1_VS
- R41 pad 1: /ChannelB2/CH_HG -> CHB2_HG
- R42 pad 1: /ChannelC1/CH_HG -> CHC1_HG
- R43 pad 1: /ChannelC2/CH_HG -> CHC2_HG
- R44 pad 2: /ChannelB2/CH_ISENSE -> CHB2_IS
- R45 pad 2: /ChannelC1/CH_ISENSE -> CHC1_IS
- R46 pad 2: /ChannelC2/CH_ISENSE -> CHC2_IS
- R47 pad 2: /ChannelB2/CH_VSENSE -> CHB2_VS
- R48 pad 2: /ChannelC1/CH_VSENSE -> CHC1_VS
- R49 pad 2: /ChannelC2/CH_VSENSE -> CHC2_VS
- R50 pad 1: /ChannelB2/CH_VSENSE -> CHB2_VS
- R51 pad 1: /ChannelC1/CH_VSENSE -> CHC1_VS
- R52 pad 1: /ChannelC2/CH_VSENSE -> CHC2_VS
- U4 pad 10: ISENSE_CHA -> CHC1_VS
- U4 pad 11: unconnected-(U4-PC3-Pad11) -> CHB2_VS
- U4 pad 12: unconnected-(U4-PA0-Pad12) -> CHB1_VS
- U4 pad 13: unconnected-(U4-PA1-Pad13) -> CHA2_VS
- U4 pad 14: unconnected-(U4-PA2-Pad14) -> CHA1_VS
- U4 pad 19: unconnected-(U4-PA5-Pad19) -> CHC2_IS
- U4 pad 20: unconnected-(U4-PA6-Pad20) -> CHC1_IS
- U4 pad 21: VSENSE_CHA -> CHB2_IS
- U4 pad 22: unconnected-(U4-PC4-Pad22) -> CHB1_IS
- U4 pad 23: unconnected-(U4-PC5-Pad23) -> CHA2_IS
- U4 pad 24: VSENSE_CHB -> unconnected-(U4-PB0-Pad24)
- U4 pad 26: unconnected-(U4-PB2-Pad26) -> CHA1_IS
- U4 pad 34: unconnected-(U4-PB12-Pad34) -> CHC2_DRVH
- U4 pad 35: VSENSE_INPUT -> CHC1_DRVH
- U4 pad 42: Net-(U4-PA8) -> CHA1_DRVH
- U4 pad 43: Net-(U4-PA9) -> CHA2_DRVH
- U4 pad 44: Net-(U4-PA10) -> CHB1_DRVH
- U4 pad 45: RGB_DATA -> CHB2_DRVH
- U4 pad 5: Net-(U4-PF0) -> unconnected-(U4-PF0-Pad5)
- U4 pad 55: unconnected-(U4-PD2-Pad55) -> BTN6
- U4 pad 56: unconnected-(U4-PB3-Pad56) -> BTN5
- U4 pad 57: unconnected-(U4-PB4-Pad57) -> RGB_DATA
- U4 pad 58: unconnected-(U4-PB5-Pad58) -> BTN4
- U4 pad 59: unconnected-(U4-PB6-Pad59) -> BTN3
- U4 pad 6: Net-(U4-PF1) -> unconnected-(U4-PF1-Pad6)
- U4 pad 60: unconnected-(U4-PB7-Pad60) -> BTN2
- U4 pad 62: unconnected-(U4-PB9-Pad62) -> BTN1
- U4 pad 8: ISENSE_INPUT -> VSENSE_INPUT
- U4 pad 9: ISENSE_CHB -> CHC2_VS
- U6 pad 12: unconnected-(U6-VS3-Pad12) -> CHB1_SW
- U6 pad 13: unconnected-(U6-HO3-Pad13) -> CHB1_HG
- U6 pad 14: unconnected-(U6-VB3-Pad14) -> Net-(D19-K)
- U6 pad 15: unconnected-(U6-VS2-Pad15) -> CHA2_SW
- U6 pad 16: unconnected-(U6-HO2-Pad16) -> CHA2_HG
- U6 pad 17: unconnected-(U6-VB2-Pad17) -> Net-(D18-K)
- U6 pad 18: CHA_SW -> CHA1_SW
- U6 pad 19: CHA_HG -> CHA1_HG
- U6 pad 22: CHA1_DRVH -> Net-(RN2-R1.2)
- U6 pad 23: CHA2_DRVH -> Net-(RN2-R2.2)
- U6 pad 24: CHB1_DRVH -> Net-(RN2-R3.2)
Other:
- board outline added: 100 x 100 mm

Commit message: layout half done
Parts:
- C1, C14, C16, C18, C53, C6, C9, L1, R1, R2, R24, R25, U3: moved to F.Cu
- C104, C105, C106, C107, C108, C109, C29, C90, D20, D21, D22, D29, D30, D31, D4, D5, D6, R64: moved to B.Cu
- moved D4 184.2 mm to (252.6, 133.3), turned to -90 degrees
- moved SW6 176.8 mm to (252.0, 131.0), turned to 90 degrees
- moved D5 174.7 mm to (252.6, 119.1), turned to -90 degrees
- moved SW5 174.6 mm to (252.0, 117.0), turned to 90 degrees
- moved C37 172.6 mm to (271.6, 63.7)
- moved SW4 172.5 mm to (252.0, 102.0), turned to 90 degrees
- moved C101 171.3 mm to (270.0, 73.5)
- moved C38 171.3 mm to (270.0, 68.5)
- moved C39 171.3 mm to (270.0, 71.0)
- moved R54 170.9 mm to (278.0, 66.0)
- moved R55 170.9 mm to (278.0, 68.5)
- moved SW3 170.9 mm to (252.0, 88.0), turned to 90 degrees
- moved C102 170.7 mm to (270.0, 76.0)
- moved C103 170.7 mm to (270.0, 78.5)
- moved R56 169.7 mm to (278.0, 71.0)
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Connections:
- C90 pad 2: +3.3V -> /VREF
- C91 pad 2: +3.3V -> /VREF
- U4 pad 28: +3.3V -> /VREF
Routing:
- net CHB1_SW: track 0.00 -> 30.3 mm, vias 0 -> 18
- net CHC2_SW: track 0.00 -> 29.5 mm, vias 0 -> 18
- net Net-(Q9-G): track 0.00 -> 27.6 mm
- net Net-(Q6-G): track 0.00 -> 25.8 mm
- net CHA1_SW: track 0.00 -> 21.1 mm, vias 0 -> 18
- net CHC1_SW: track 0.00 -> 20.0 mm, vias 0 -> 18
- net CHA2_SW: track 0.00 -> 19.2 mm, vias 0 -> 18
- net Net-(Q8-G): track 0.00 -> 18.6 mm
- net Net-(Q4-G): track 0.00 -> 17.7 mm
- net Net-(Q5-G): track 0.00 -> 16.7 mm
- net CHB2_SW: track 0.00 -> 16.4 mm, vias 0 -> 18
- net Net-(Q7-G): track 0.00 -> 15.6 mm
- net CHC2_IS: track 0.00 -> 9.21 mm
- net CHB1_IS: track 0.00 -> 7.87 mm
- net CHA1_IS: track 0.00 -> 6.82 mm
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- added copper zone on F.Cu, net /ChannelA1/CH_VOUT
- added copper zone on F.Cu, net /ChannelA2/CH_VOUT
- added copper zone on F.Cu, net /ChannelB1/CH_VOUT
- added copper zone on F.Cu, net /ChannelB2/CH_VOUT
- added copper zone on F.Cu, net /ChannelC1/CH_VOUT
- added copper zone on F.Cu, net /ChannelC2/CH_VOUT
- added copper zone on F.Cu, net CHA1_SW
- added copper zone on F.Cu, net CHA2_SW
- added copper zone on F.Cu, net CHB1_SW
- added copper zone on F.Cu, net CHB2_SW
- added copper zone on F.Cu, net CHC1_SW
- added copper zone on F.Cu, net CHC2_SW
- added copper zone on F.Cu, net GNDPWR
- added copper zone on B.Cu, net Net-(C59-Pad1)
- added copper zone on F.Cu, net Net-(C59-Pad1)
- added copper zone on B.Cu, net Net-(C63-Pad1)
- added copper zone on F.Cu, net Net-(C63-Pad1)
- added copper zone on B.Cu, net Net-(C69-Pad1)
- added copper zone on F.Cu, net Net-(C69-Pad1)
- added copper zone on B.Cu, net Net-(C92-Pad1)
- added copper zone on F.Cu, net Net-(C92-Pad1)
- added copper zone on B.Cu, net Net-(C93-Pad1)
- added copper zone on F.Cu, net Net-(C93-Pad1)
- added copper zone on B.Cu, net Net-(C94-Pad1)
- added copper zone on F.Cu, net Net-(C94-Pad1)
- added copper zone on F.Cu, net Net-(J10-Pin_1)
- added copper zone on F.Cu, net Net-(J3-Pin_1)
- added copper zone on F.Cu, net Net-(J4-Pin_1)
- added copper zone on F.Cu, net Net-(J5-Pin_1)
- added copper zone on F.Cu, net Net-(J6-Pin_1)
- added copper zone on F.Cu, net Net-(J9-Pin_1)
- added copper zone on F.Cu, net VPP
- removed copper zone on In2.Cu, net +10V
- removed copper zone on F.Cu, net +3.3V
- removed copper zone on In2.Cu, net +3.3V
- removed copper zone on In2.Cu, net +5V
- removed copper zone on B.Cu, net GND
- removed copper zone on F.Cu, net GND
- removed copper zone on In1.Cu, net GND
- removed copper zone on In2.Cu, net VPP
Other:
- board text removed: "I_A"
- board text removed: "I_B"
- board text removed: "I_IN"
- board text removed: "V_A"
